File: pcb/backups/pre stitch 3.kicad_pcb (KiCad board)
At the start: 2 copper layers, 50 x 99 mm, 40 parts, among them J1 Conn_01x04, J2 Conn_01x05, J3 Conn_01x02, SW1 SW_PUSH, U1 STM32F072CBTx, U2 TLV75533PDBV

Commit message: added reset switches
Routing:
- net GND: vias 945 -> 30
