File: pcb/joy.kicad_pcb (KiCad board)
At the start: 2 copper layers, 50 x 99 mm, 40 parts, among them J1 Conn_01x04, J2 Conn_01x05, J3 Conn_01x02, SW1 SW_PUSH, U1 STM32F072CBTx, U2 TLV75533PDBV

Commit message: added switches, redid routing, updated pins
Parts:
- removed J3: Conn_01x02, Connector_PinHeader_2.54mm:PinHeader_1x02_P2.54mm_Vertical
- added BOOT0: SW_PUSH, Button_Switch_SMD:SW_SPST_SKQG_WithStem, F.Cu at (6.90, 24.9)
- moved R10 7.42 mm to (3.80, 29.8)
- renumbered SW1 to NRST
Routing:
- net BOOT0: track 9.61 -> 23.3 mm
- net +3V3: track 132.1 -> 145.7 mm
- net GND: track 73.1 -> 78.2 mm, vias 945 -> 323
- net MF1COM: track 80.0 -> 79.9 mm, vias 1 -> 2
- net MF1PUSH: vias 1 -> 2
- net MF1D: vias 1 -> 2
